File: schematPCB/schemat.brd (EAGLE design)
At the start: 160 x 100 mm, 33 parts, among them IC1 MEGA8-P, IC2 L293D

Commit message: prawidlowe schematy
Parts:
- moved C7 134.5 mm to (87.1, 61.3)
- moved C2 122.5 mm to (67.3, 57.1), turned to 90 degrees
- moved C6 118.4 mm to (73.4, 79.8), turned to 90 degrees
- moved C5 113.1 mm to (87.1, 55.8), turned to 270 degrees
- moved C1 111.3 mm to (63.5, 55.9), turned to 90 degrees
- moved C3 110.6 mm to (48.3, 57.1), turned to 270 degrees
- moved C4 99.5 mm to (69.2, 79.8), turned to 90 degrees
- moved LED2 98.3 mm to (35.7, 78.2), turned to 90 degrees
- moved LED1 97.9 mm to (41.7, 78.2), turned to 90 degrees
- moved L1 95.8 mm to (70.2, 53.3), turned to 180 degrees
- moved ENKODER2 87.1 mm to (38.6, 57.9)
- moved R1 84.8 mm to (48.4, 71.4), turned to 90.8 degrees
- moved ENKODER1 77.6 mm to (38.6, 64.6)
- moved R6 70.7 mm to (42.5, 70.9), turned to 180.1 degrees
- moved RASPBERRY 65.3 mm to (82.5, 55.9), turned to 270 degrees
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Connections:
- removed net GNDEL: C1.2, C2.2, C3.2, ENKODER1.2, ENKODER2.2, HV.4, IC1.22, IC1.8, LED1.2, LED2.2, P-EL-OUT.2, RASPBERRY.2
- removed net GNDS: P-S-OUT.2, SERWO1.3, SERWO2.3, SERWO3.3
- net GND: now also C1.2, C2.2, C3.2, ENKODER1.2, ENKODER2.2, HV.4, IC1.22, IC1.8, LED1.2, LED2.2, P-EL-OUT.2, P-S-OUT.2, RASPBERRY.2, SERWO1.3, SERWO2.3, SERWO3.3
Routing:
- net GND: track 0.00 -> 209.0 mm, vias 0 -> 2
- net +5V: track 0.00 -> 114.0 mm, vias 0 -> 2
- net SILNIK1_PWM: track 0.00 -> 87.5 mm
- net SILNIK2_PWM: track 0.00 -> 83.9 mm, vias 0 -> 2
- net RESET: track 0.00 -> 52.2 mm, vias 0 -> 2
- net SS: track 0.00 -> 43.1 mm
- net VCC: track 0.00 -> 32.9 mm
- net SILNIK2_1: track 0.00 -> 30.4 mm
- net SILNIK1_1: track 0.00 -> 29.6 mm, vias 0 -> 2
- net ENKODER1: track 0.00 -> 18.6 mm, vias 0 -> 2
- net SILNIK2_2: track 0.00 -> 16.4 mm
- net V+: track 0.00 -> 16.4 mm
- net SILNIK1_2: track 0.00 -> 15.7 mm
- net ENKODER1_I: track 0.00 -> 15.1 mm
- net ENKODER2_I: track 0.00 -> 14.9 mm
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- added copper zone on layer 16, net GND
Other:
- board size 160 x 100 mm -> 63.2 x 56.8 mm
