File: schematPCB/schemat.sch (EAGLE design)
At the start: 33 parts, among them IC1 MEGA8-P, IC2 L293D

Commit message: prawidlowe schematy
Connections:
- removed net GNDEL: C1.2, C2.2, C3.2, ENKODER1.2, ENKODER2.2, HV.4, IC1.GND, IC1.GND@1, LED1.2, LED2.2, P-EL-OUT.2, RASPBERRY.2
- removed net GNDS: P-S-OUT.2, SERWO1.3, SERWO2.3, SERWO3.3
- net GND: now also C1.2, C2.2, C3.2, ENKODER1.2, ENKODER2.2, HV.4, IC1.GND, IC1.GND@1, LED1.2, LED2.2, P-EL-OUT.2, P-S-OUT.2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
